File: Transformer driver/current voltage.kicad_sch (KiCad schematic)
At the start: 6 parts, among them U2 LM311, U3 4047, U4 LM393

Commit message: another one commit
Parts:
- added D5: LED, symbol Device:LED
- added R11: R, symbol Device:R
Connections:
- new net: D5.1 (K), R11.2
- new net +5V: R11.1
