File: Transformer driver/MA_LED.kicad_sch (KiCad schematic)
At the start: 8 parts, among them Q8 IRF540N, U6 LM311, U8 74HC74

Commit message: commit
Parts:
- removed R22: R, symbol Device:R
- added C11, C12, C13, C14: C, symbol Device:C
- added R26, R27: R, symbol Device:R
- added RV1: R_Potentiometer, symbol Device:R_Potentiometer
- added U7: 74AHC1G00, symbol 74xGxx:74AHC1G00
Connections:
- net +15V: now also R26.1, U7.5 (VCC)
- net GND: now also C11.2, C12.2, C13.2, C14.2, RV1.3, U7.3 (GND)
- net at R25.2, U6.7, U8.3 (C): now also C11.1
- net at R21.1: now also RV1.1; no longer U6.3 (-)
- net at U8.4 (~{S}): now also U7.4
- new net: C12.1, C13.1, R27.2
- new net: C14.1, RV1.2, U6.3 (-)
- new net RESET: R26.2, R27.1, U7.1, U7.2
- no-connect marks 0 -> 1
Other:
- moved on the sheet: D6, Q8, R21, R24, R25, U6, U8A
