File: Transformer driver/ma side.kicad_sch (KiCad schematic)
At the start: 8 parts, among them Q1 NPN, Q3 NPN, Q4 PNP, Q5 PNP, Q6 IRF540N, Q7 IRF540N, U5 IR2153

Commit message: more commits for mA
Parts:
- added C6: C, symbol Device:C
- added R12: R, symbol Device:R
- added R13: 0.20m, symbol Device:R
Connections:
- net +15V: now also U5.1 (VCC), U5.8 (VB)
- net GND: now also U5.4 (COM), U5.6 (VS), C6.2
- net at Q7.2 (D): now also TR1.6
- net at Q7.3 (S): now also Q6.3 (S), R13.1
- net +48v: now reaches TR1.1
- net +48v: now also TR1.4
- net at TR1.3: now also Q6.2 (D)
- net at U5.2 (RT): now also R12.1
- net at U5.3 (CT): now also C6.1, R12.2
- new net -48v: R13.2
Other:
- moved on the sheet: TR1

Commit message: commit more changes
Parts:
- added C7: C, symbol Device:C
- added R14, R15, R16, R17, R18: R, symbol Device:R
Connections:
- net at Q3.3 (E), Q5.3 (E): now also R15.1; no longer Q7.1 (G)
- net at Q3.2 (B), Q5.2 (B): now also R17.1; no longer U5.5 (LO)
- net at Q1.2 (B), Q4.2 (B): now also R16.2; no longer U5.7 (HO)
- net at Q1.3 (E), Q4.3 (E): now also R14.1; no longer Q6.1 (G)
- net at TR1.10: now also TR1.9
- net at Q6.2 (D), TR1.3: now also R18.1
- new net: R16.1, U5.7 (HO)
- new net: Q7.1 (G), R15.2
- new net: C7.1, R18.2
- new net: Q6.1 (G), R14.2
- new net: R17.2, U5.5 (LO)

Commit message: adding documents
Parts:
- added C8: C, symbol Device:C
- added R19: R, symbol Device:R
Connections:
- net -48v: now also C7.2, TR1.12, C8.2
- net at Q7.2 (D), TR1.6: now also R19.1
- new net: C8.1, R19.2
Other:
- moved on the sheet: C7, R17, R18

Commit message: more on the ma side
Parts:
- added C10, C9: C, symbol Device:C
- added R20, R23: R, symbol Device:R
Connections:
- net GND: now also C10.2, C9.2, R23.1
- net at Q6.3 (S), Q7.3 (S), R13.1: now also C10.1, C9.1, R20.1
- new net Imeasure: R20.2, R23.2
Other:
- added sheet mA alarm indicator (MA_LED.kicad_sch)
- moved on the sheet: C6, C7, C8, Q1, Q3, Q4, Q5, Q6, Q7, R12, R13, R14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

Commit message: commit
Parts:
- added C15: C, symbol Device:C
- added C16: C_Polarized, symbol Device:C_Polarized
Connections:
- net +15V: now also C15.1, C16.1
- net GND: now also C15.2, C16.2
Other:
- moved on the sheet: C10, C9, R20, R23
