File: Transformer driver/untitled.kicad_sch (KiCad schematic)
At the start: 0 parts

Commit message: commits
Changed lines of the file:
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@@
 		(exclude_from_sim no)
 		(at 17.78 19.05 0)
-		(size 201.93 11.43)
+		(size 224.79 16.51)
 		(margins 0.9525 0.9525 0.9525 0.9525)
 		(stroke
@@
 			(font
 				(size 2.54 2.54)
+				(thickness 0.508)
+				(bold yes)
 			)
 			(justify left top)
+		)
+	)
+	(text_box "From the Op amp the signal must go to a latch like the IC on the channel card."
+		(exclude_from_sim no)
+		(at 17.78 36.83 0)
+		(size 223.52 19.05)
+		(margins 0.9525 0.9525 0.9525 0.9525)
+		(stroke
+			(width 0)
+			(type solid)
+		)
+		(fill
+			(type none)
+		)
+		(effects
+			(font
+				(size 2.54 2.54)
+				(thickness 0.508)
+				(bold yes)
+			)
+			(justify left top)

Commit message: commit more changes
Other:
- note added: "Fron when the signal comes from the shunt resistor it goes though a lot of curcuitry that might be there for protection because zener diodes are there."
- note added: "R13=200mOhm shunt resistor"
Changed lines of the file:
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@@
 	(generator_version "9.0")
 	(paper "A4")
+	(text "R13=200mOhm shunt resistor"
+		(exclude_from_sim no)
+		(at 51.054 63.754 0)
+		(effects
+			(font
+				(size 2.54 2.54)
+				(thickness 0.508)
+				(bold yes)
+			)
+		)
+	)
+	(text "Fron when the signal comes from the shunt resistor it goes \nthough a lot of curcuitry that might be there for protection\n because zener diodes are there."
+		(exclude_from_sim no)
+		(at 78.74 81.026 0)
+		(effects
+			(font
+				(size 2.54 2.54)
+				(thickness 0.254)
+				(bold yes)
+			)
+		)
+	)
 	(text_box "THE IGBT MODULE VERSION IS GAL DO NOT BE CONFUSED WHEN YOU SEE A MODULE WITH TWO IGBTS."
 		(exclude_from_sim no)

Commit message: more on the ma side
Other:
- note added: "All the resistor on a potential divider for input comparators are to be potentiometers to adjust the level at which the alarms are triggered."
Changed lines of the file:
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@@
 	(generator_version "9.0")
 	(paper "A4")
+	(text "All the resistor on a potential divider for input\n comparators are to be potentiometers\n to adjust the level at which the alarms are triggered."
+		(exclude_from_sim no)
+		(at 70.358 101.346 0)
+		(effects
+			(font
+				(size 2.54 2.54)
+				(thickness 0.508)
+				(bold yes)
+			)
+		)
+	)
 	(text "R13=200mOhm shunt resistor"
 		(exclude_from_sim no)
@@
 		(effects
 			(font
+				(face "KiCad Font")
 				(size 2.54 2.54)
 				(thickness 0.254)

Commit message: commit
Other:
- note added: "The primary shunt detects overcurrent due to core saturation. The output will detect overcurrent due to faulty XRT."
- note added: "lIST iCS THAT WORK ON 5v AND THOSE THAT WORK ON 15v"
Changed lines of the file:
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@@
 	(generator_version "9.0")
 	(paper "A4")
+	(text "lIST iCS THAT WORK ON 5v AND THOSE THAT WORK ON 15v"
+		(exclude_from_sim no)
+		(at 76.2 131.826 0)
+		(effects
+			(font
+				(size 2.54 2.54)
+				(thickness 0.254)
+				(bold yes)
+			)
+		)
+	)
 	(text "All the resistor on a potential divider for input\n comparators are to be potentiometers\n to adjust the level at which the alarms are triggered."
 		(exclude_from_sim no)
 		(at 70.358 101.346 0)
+		(effects
+			(font
+				(size 2.54 2.54)
+				(thickness 0.508)
+				(bold yes)
+			)
+		)
+	)
+	(text "The primary shunt detects overcurrent due to core saturation.\nThe output will detect overcurrent due to faulty XRT."
+		(exclude_from_sim no)
+		(at 78.74 119.126 0)
 		(effects
 			(font
@@
 		(effects
 			(font
-				(face "KiCad Font")
 				(size 2.54 2.54)
 				(thickness 0.254)
